File: LickSensor_EAGLE_FILES_COPY/LickSensor_V3.brd (EAGLE design)
At the start: 68.6 x 53.3 mm, 50 parts, among them Q1 IRL540NPBF, Q2 IRL540NPBF, T1 BC547, T2 BC547, U1 ARDUINOR3-DIMENSION

Commit message: updated eagle files
Parts:
- R6: value 1M -> 10k
Changed lines of the file:
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@@
 <attribute name="VALUE" x="-43.688" y="24.384" size="1.27" layer="27" ratio="10" rot="R180"/>
 </element>
-<element name="R6" library="rcl" library_urn="urn:adsk.eagle:library:334" package="0204/7" package3d_urn="urn:adsk.eagle:package:23498/2" value="1M" x="-41.91" y="29.21" smashed="yes" rot="R270">
+<element name="R6" library="rcl" library_urn="urn:adsk.eagle:library:334" package="0204/7" package3d_urn="urn:adsk.eagle:package:23498/2" value="10k" x="-41.91" y="29.21" smashed="yes" rot="R270">
 <attribute name="NAME" x="-40.6146" y="31.75" size="0.8128" layer="25" ratio="10" rot="R270"/>
 <attribute name="SPICEPREFIX" value="R" x="-41.91" y="29.21" size="1.778" layer="27" rot="R270" display="off"/>
@@
 </element>
 <element name="LICK_IN_PAD" library="testpad" library_urn="urn:adsk.eagle:library:385" package="P1-13" package3d_urn="urn:adsk.eagle:package:27946/1" value="TPPAD1-13" x="-21.59" y="46.99" smashed="yes">
-<attribute name="NAME" x="-22.606" y="48.26" size="0.8128" layer="25" ratio="10"/>
+<attribute name="NAME" x="-23.876" y="48.26" size="0.8128" layer="25" ratio="10"/>
 <attribute name="TP_SIGNAL_NAME" value="" x="-21.59" y="46.99" size="1.778" layer="27" display="off"/>
 <attribute name="VALUE" x="-21.59" y="46.99" size="0.0254" layer="27"/>
@@
 </element>
 <element name="GNDPINS" library="adafruit" library_urn="urn:adsk.eagle:library:420" package="1X03" package3d_urn="urn:adsk.eagle:package:6240710/1" value="" x="-73.66" y="52.07" smashed="yes">
-<attribute name="NAME" x="-77.5462" y="53.8988" size="0.8128" layer="25" ratio="10"/>
+<attribute name="NAME" x="-75.7682" y="49.0728" size="0.8128" layer="25" ratio="10"/>
 <attribute name="VALUE" x="-77.47" y="48.895" size="1.27" layer="27"/>
 </element>
@@
 </element>
 <element name="LICKIN_GND" library="adafruit" package="1X01" value="" x="-21.59" y="44.45" smashed="yes">
-<attribute name="NAME" x="-22.9362" y="46.2788" size="1.27" layer="25" ratio="10"/>
+<attribute name="NAME" x="-24.4602" y="41.9608" size="0.6096" layer="25" ratio="10"/>
 <attribute name="VALUE" x="-22.86" y="41.275" size="1.27" layer="27"/>
 </element>
